Commit message: slam_working

File: bramm_description/urdf/bramm.xacro (robot description, xacro)
@@ -4,4 +4,5 @@
 <xacro:include filename="$(find bramm_description)/urdf/bramm.trans" />
 <xacro:include filename="$(find bramm_description)/urdf/bramm.gazebo" />
+<link name="base_footprint"/>
 <link name="base_link">
  <inertial>
@@ -167,4 +168,33 @@
   </collision>
 </link>
+<gazebo reference="lidar_1">
+  <sensor type="ray" name="lidar_sensor">
+    <visualize>true</visualize>
+    <update_rate>20</update_rate>
+    <ray>
+      <scan>
+        <horizontal>
+          <samples>720</samples>
+          <resolution>1</resolution>
+          <min_angle>-3.14159</min_angle>
+          <max_angle>3.14159</max_angle>
+        </horizontal>
+      </scan>
+      <range>
+        <min>0.12</min>
+        <max>20.0</max>
+        <resolution>0.01</resolution>
+      </range>
+    </ray>
+    <plugin name="gazebo_ros_laser" filename="libgazebo_ros_ray_sensor.so">
+  <ros>
+    <remapping>~/out:=scan</remapping>
+  </ros>
+  <frame_name>lidar_1</frame_name>
+  <topic_name>scan</topic_name>
+  <output_type>sensor_msgs/LaserScan</output_type>
+</plugin>
+  </sensor>
+</gazebo>
 <link name="camera_1">
   <inertial>
@@ -251,17 +281,22 @@
   </collision>
 </link>
-<joint name="right_wheel_joint" type="continuous">
+<joint name="base_footprint_joint" type="fixed">
+  <parent link="base_footprint"/>
+  <child link="base_link"/>
+  <origin xyz="0 0 0" rpy="0 0 0"/>
+</joint>
+<joint name="Revolute 3" type="continuous">
   <origin xyz="-0.09 -0.05 0.0025" rpy="0 0 0"/>
   <parent link="base_link"/>
   <child link="wheel_rr_1"/>
-  <axis xyz="0.0 1.0 0.0"/>
-</joint>
-<joint name="left_wheel_joint" type="continuous">
+  <axis xyz="0 1 0"/>
+</joint>
+<joint name="Revolute 7" type="continuous">
   <origin xyz="-0.09 0.05 0.0025" rpy="0 0 0"/>
   <parent link="base_link"/>
   <child link="wheel_rl_1"/>
-  <axis xyz="0.0 1.0 0.0"/>
-</joint>
-<joint name="elbo_joint" type="continuous">
+  <axis xyz="0 1 0"/>
+</joint>
+<joint name="Revolute 8" type="continuous">
   <origin xyz="0.074661 0.01555 0.023" rpy="0 0 0"/>
   <parent link="base_link"/>
@@ -269,5 +304,5 @@
   <axis xyz="0.0 -1.0 0.0"/>
 </joint>
-<joint name="arm_joint" type="continuous">
+<joint name="Revolute 9" type="continuous">
   <origin xyz="0.0 -0.006 0.115" rpy="0 0 0"/>
   <parent link="elbo_1_1"/>
@@ -275,15 +310,15 @@
   <axis xyz="0.0 -1.0 0.0"/>
 </joint>
-<joint name="Rigid_1" type="fixed">
+<joint name="Rigid 11" type="fixed">
   <origin xyz="-0.09 0.0 0.005" rpy="0 0 0"/>
   <parent link="base_link"/>
   <child link="lidar_stand_1"/>
 </joint>
-<joint name="Rigid_2" type="fixed">
-  <origin xyz="0.0 0.0 0.17" rpy="0 0 0"/>
+<joint name="Rigid 12" type="fixed">
+  <origin xyz="0.0 0.0 0.175" rpy="0 0 0"/>
   <parent link="lidar_stand_1"/>
   <child link="lidar_1"/>
 </joint>
-<joint name="Rigid_3" type="fixed">
+<joint name="Rigid 13" type="fixed">
   <origin xyz="-0.015 0.013 0.205" rpy="0 0 0"/>
   <parent link="arm_1_1"/>
@@ -316,10 +351,10 @@
     <plugin>gazebo_ros2_control/GazeboSystem</plugin>
   </hardware>
-  <joint name="left_wheel_joint">
+  <joint name="Revolute 7">
     <command_interface name="velocity"/>
     <state_interface name="velocity"/>
     <state_interface name="position"/>
   </joint>
-  <joint name="right_wheel_joint">
+  <joint name="Revolute 3">
     <command_interface name="velocity"/>
     <state_interface name="velocity"/>

Commit message: adding vision node

File: bramm_description/urdf/bramm.xacro (robot description, xacro)
@@ -218,4 +218,27 @@
   </collision>
 </link>
+<gazebo reference="camera_1">
+  <sensor type="camera" name="camera">
+    <update_rate>30</update_rate>
+      <camera>
+        <horizontal_fov>1.047</horizontal_fov>
+        <image>
+          <width>640</width>
+          <height>480</height>
+          <format>R8G8B8</format>
+        </image>
+        <clip>
+          <near>0.1</near>
+          <far>100.0</far>
+        </clip>
+      </camera>
+    <plugin name="camera_controller" filename="libgazebo_ros_camera.so">
+      <camera_name>camera</camera_name>
+      <image_topic_name>image_raw</image_topic_name>
+      <camera_info_topic_name>camera_info</camera_info_topic_name>
+      <frame_name>camera_link</frame_name>
+    </plugin>
+  </sensor>
+</gazebo>
 <link name="camera2_1">
   <inertial>
@@ -239,4 +262,27 @@
   </collision>
 </link>
+<gazebo reference="camera2_1">
+  <sensor type="camera" name="camera2">
+    <update_rate>30</update_rate>
+      <camera>
+        <horizontal_fov>1.047</horizontal_fov>
+        <image>
+          <width>640</width>
+          <height>480</height>
+          <format>R8G8B8</format>
+        </image>
+        <clip>
+          <near>0.1</near>
+          <far>100.0</far>
+        </clip>
+      </camera>
+    <plugin name="camera_controller2" filename="libgazebo_ros_camera.so">
+      <camera_name>camera2</camera_name>
+      <image_topic_name>image_raw2</image_topic_name>
+      <camera_info_topic_name>camera_info2</camera_info_topic_name>
+      <frame_name>camera_link2</frame_name>
+    </plugin>
+  </sensor>
+</gazebo>
 <link name="gripper_left_1">
   <inertial>
@@ -260,4 +306,5 @@
   </collision>
 </link>
+Therefore
 <link name="gripper_right_1">
   <inertial>
@@ -314,4 +361,5 @@
   <parent link="base_link"/>
   <child link="lidar_stand_1"/>
+Therefore
 </joint>
 <joint name="Rigid 12" type="fixed">
@@ -351,4 +399,5 @@
     <plugin>gazebo_ros2_control/GazeboSystem</plugin>
   </hardware>
+  <!-- wheels -->
   <joint name="Revolute 7">
     <command_interface name="velocity"/>
@@ -361,4 +410,13 @@
     <state_interface name="position"/>
   </joint>
+  <!-- arm -->
+  <joint name="Revolute 8">
+    <command_interface name="position"/>
+    <state_interface name="position"/>
+  </joint>
+  <joint name="Revolute 9">
+    <command_interface name="position"/>
+    <state_interface name="position"/>
+  </joint>
 </ros2_control>
 <gazebo reference="wheel_rl_1">
